File: HW/meracia_jednotka_v1.kicad_sch (KiCad schematic)
At the start: 31 parts, among them IC1 MAX77827CEFD+T, J1 microSD Reader, J2 LoRa digital, J3 DS18B20, J4 DS18B20, J5 DS18B20, J7 DS18B20, J8 DS18B20, J9 DS18B20, U1 Ai-Thinker-Ra-02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

Commit message: Add files via upload
LDO added
Parts:
- removed C10, C11, C9: C, symbol Device:C
- removed L2: L, symbol Device:L
- removed R5, R6: R, symbol Device:R
- removed U2: TLV62569DBV, Package_TO_SOT_SMD:SOT-23-5, symbol Regulator_Switching:TLV62569DBV
- added U2: AZ1117-3.3, symbol Regulator_Linear:AZ1117-3.3
- added U3: TPL5111, Package_TO_SOT_SMD:SOT-23-6, symbol Timer:TPL5111
- added U4: SiP32431DR3, Package_TO_SOT_SMD:SOT-363_SC-70-6, symbol Power_Management:SiP32431DR3
Connections:
- new net: U4.2 (GND), U4.5 (GND)
Other:
- note added: "5V to 3V3 LDO"
- note removed: "5V to 3V3 Buck"
- note removed: "doplniť"
- note removed: "treba ešte dopočítať súčiastky podľa datasheetu"

Commit message: Add files via upload
layout update
Parts:
- removed BT2: Battery_Cell, symbol Device:Battery_Cell
- removed C8: 1uF/25V, symbol Device:C
- removed IC1: MAX77827CEFD+T, MAX77827CEFDT, symbol MAX77827CEFD+T:MAX77827CEFD+T
- removed J2: LoRa digital, Connector_PinHeader_2.54mm:PinHeader_1x06_P2.54mm_Vertical, symbol Connector_Generic:Conn_01x06
- removed U3: TPL5111, Package_TO_SOT_SMD:SOT-23-6, symbol Timer:TPL5111
- removed U4: SiP32431DR3, Package_TO_SOT_SMD:SOT-363_SC-70-6, symbol Power_Management:SiP32431DR3
- added C10: 22uF, Capacitor_SMD:C_1206_3216Metric_Pad1.33x1.80mm_HandSolder, symbol Device:C
- added C12, C9: 1uF, Capacitor_SMD:C_0805_2012Metric_Pad1.18x1.45mm_HandSolder, symbol Device:C
- added C13: 1uF/25V, Capacitor_SMD:C_0805_2012Metric_Pad1.18x1.45mm_HandSolder, symbol Device:C
- added D2: D_Zener_Filled, Diode_SMD:D_1206_3216Metric_Pad1.42x1.75mm_HandSolder, symbol Device:D_Zener_Filled
- added R4: 10k, Resistor_SMD:R_1206_3216Metric_Pad1.30x1.75mm_HandSolder, symbol Device:R
- added R5: 100k, Resistor_SMD:R_1206_3216Metric_Pad1.30x1.75mm_HandSolder, symbol Device:R
- added U5: LV2862YDDC, Package_TO_SOT_SMD:SOT-23-6, symbol Regulator_Switching:LV2862YDDC
- C1, C2: footprint (none) -> Capacitor_SMD:C_1206_3216Metric_Pad1.33x1.80mm_HandSolder
- C3: value 22uF/25V -> 2.2uF/25V; footprint (none) -> Capacitor_SMD:C_1206_3216Metric_Pad1.33x1.80mm_HandSolder
- C4, C6: value 10uF/25V -> 10uF; footprint (none) -> Capacitor_SMD:C_1206_3216Metric_Pad1.33x1.80mm_HandSolder
- C5: value 22uF/25V -> 100nF/25V; footprint (none) -> Capacitor_SMD:C_1206_3216Metric_Pad1.33x1.80mm_HandSolder
- C7: value 1uF/25V -> 10uF/25V; footprint (none) -> Capacitor_SMD:C_1206_3216Metric_Pad1.33x1.80mm_HandSolder
- J3, J4, J5, J7, J8, J9: footprint (none) -> Connector_PinHeader_2.54mm:PinHeader_1x03_P2.54mm_Vertical
- L1: value 1uH -> 22uH; footprint (none) -> Inductor_SMD:L_Murata_LQH55DN_5.7x5.0mm
- R1, R2: footprint (none) -> Resistor_SMD:R_1206_3216Metric_Pad1.30x1.75mm_HandSolder
- R3: value 4.99k -> 54.9k; footprint (none) -> Resistor_SMD:R_1206_3216Metric_Pad1.30x1.75mm_HandSolder
- U2: footprint (none) -> Package_TO_SOT_SMD:SOT-223-3_TabPin2
Connections:
- net CSS_SD: now also J1.6 (Pin_6); no longer J1.1 (Pin_1)
- net DQ: now also A1.8 (D5)
- net GND: now also J1.1 (Pin_1), U2.1 (GND), C10.2, C12.2, C13.2, C9.2, D2.2 (A), R4.1, U5.2 (GND); no longer C5.2, J1.6 (Pin_6), R3.2
- net LORA_DIO0: now also A1.21 (A2); no longer A1.19 (A0)
- net LORA_DIO1: now also A1.22 (A3); no longer A1.20 (A1)
- net LORA_DIO2: now also A1.23 (A4); no longer A1.21 (A2)
- net LORA_DIO3: now also A1.24 (A5); no longer A1.22 (A3)
- net LORA_DIO4: now also A1.19 (A0); no longer A1.23 (A4)
- net LORA_DIO5: now also A1.20 (A1); no longer A1.24 (A5)
- net MISO: now also J1.3 (Pin_3); no longer J1.4 (Pin_4)
- net MOSI: now also J1.4 (Pin_4); no longer J1.3 (Pin_3)
- net SCK: now also J1.5 (Pin_5); no longer J1.2 (Pin_2)
- net VDD_3V3: now also C6.1, U2.2 (VO), C10.1, C12.1
- net VDD_5V: now also C4.1, J1.2 (Pin_2), L1.2, R3.2, U2.3 (VI), C9.1; no longer C5.1, C6.1, J1.5 (Pin_5)
- net at L1.1: now also C5.2, D2.1 (K), U5.6 (SW)
- net power_done: now reaches A1.12 (D9)
- net at R3.1: now also R4.2, U5.3 (FB)
- net VBAT: now reaches C3.1
- net VBAT: now also C13.1, R5.1, U5.5 (VIN); no longer C4.1
- new net: R5.2, U5.4 (~{SHDN})
- new net: C5.1, U5.1 (CB)
- no-connect marks 7 -> 13
Other:
- added sheet Power (Power.kicad_sch)
- note removed: "Nie je nutné, pre istotu som to vyviedla aj na piny"
- moved on the sheet: C3, C5, J1, L1
